Commit message: v3.0 更改模型文件

File: src/assets/e1_21dof/urdf/E1_21dof.urdf (robot description, URDF)
Before this commit: robot E1_2_v1, 28 links, 27 joints
Links:
- link left_hip_pitch_link: mass 1.01 -> 1.334; geometry collision mesh filename=../meshes/left_hip_pitch_link_v1.STL; visual mesh filename=../meshes/left_hip_pitch_link_v1.STL
- link left_hip_roll_link: geometry collision mesh filename=../meshes/left_hip_roll_link_v1.STL; visual mesh filename=../meshes/left_hip_roll_link_v1.STL
- link right_hip_pitch_link: mass 1.005 -> 1.334; geometry collision mesh filename=../meshes/right_hip_pitch_link_v1.STL; visual mesh filename=../meshes/right_hip_pitch_link_v1.STL
- link right_hip_roll_link: geometry collision mesh filename=../meshes/right_hip_roll_link_v1.STL; visual mesh filename=../meshes/right_hip_roll_link_v1.STL
Joints:
- joint left_hip_roll_joint: limit lower=-0.5236 upper=3.1416 effort=60 velocity=13.09 -> lower=-0.5236 upper=3.1416 effort=120 velocity=12.04; origin xyz=0 0.0625 -0.02 rpy=0 0 0 -> xyz=0 0.0725 -0.012 rpy=0 0 0
- joint left_hip_yaw_joint: origin xyz=0 0.01 -0.098 rpy=0 0 0 -> xyz=0 0 -0.106 rpy=0 0 0
- joint right_hip_roll_joint: limit lower=-3.1416 upper=0.5236 effort=60 velocity=13.09 -> lower=-3.1416 upper=0.5236 effort=120 velocity=12.04; origin xyz=0 -0.0625 -0.02 rpy=0 0 0 -> xyz=0 -0.0725 -0.012 rpy=0 0 0
- joint right_hip_yaw_joint: origin xyz=0 -0.01 -0.098 rpy=0 0 0 -> xyz=0 0 -0.106 rpy=0 0 0
